File: PIC795 Brain Board.brd (EAGLE design)
At the start: 127 x 88.9 mm, 56 parts, among them J10 MOLEX_4PMOLEX_4P, J11 MOLEX_6P, J12 MOLEX_3P, J13 MOLEX-2P-156, J5 MOLEX_4PMOLEX_4P, J6 MOLEX_4PMOLEX_4P, J7 USB+SHIELD, J8 POWER_JACK, J9 RJ11-2L-B, SW1 E_SWITCH-320, U1 REGULATOR_LD1086_LDO, U2 SD_CARD, U3 PIC32MX795F512L, U4 MAX4830, U5 24LC256, X1 8 Mhz

Commit message: Add files via upload
Minor changes for Rev 2
Parts:
- D1, D2: value 1N5817-B -> 40V
- LED1: value (none) -> RED
- LED2: value (none) -> YELLOW
- R1, R3: value 120 ohm -> 220 ohm
- moved J9 0.63 mm to (66.0, 4.45)
Connections:
- net !SD_CS renamed T5CK
- net GND: no longer J1.25, J1.26
Other:
- board text added: "+5V"
- board text added: "ROBOTNIK BRAIN BOARD REV 2"
- board text removed: "ROBOTNIK BRAIN BOARD REV 1"

Commit message: Add files via upload
Includes latest changes for Rev 2. Shipped to PCB fab 8-12-19
Parts:
- added CS, MISO, MOSI, SCK: TP, JimLib:TESTPAD
- added J14: MOLEX_MINI_RA_3P, JimLib:MOLEX_MINI_RA_3P
- added J15: MOLEX_4PMOLEX_4P, JimLib:MOLEX_4P
- added J16: (no value), JimLib:2X7
- added R4, R5: 10K, JimLib:1/4_WATT
- added R6: 180 ohms, JimLib:0204/7
- moved GNDB 19.6 mm to (6.12, 72.9)
- moved C20 9.68 mm to (63.6, 83.9), turned to 180 degrees
- moved C10 8.53 mm to (69.4, 54.0), turned to 90 degrees
- moved C8 6.38 mm to (61.0, 54.0), turned to 90 degrees
- moved C11 6.35 mm to (54.0, 50.8), turned to 0 degrees
- moved C5 5.38 mm to (66.4, 34.9), turned to 270 degrees
- moved J11 5.34 mm to (46.0, 6.10), turned to 0 degrees
- moved C9 5.24 mm to (66.0, 54.0), turned to 90 degrees
- moved C3 5.12 mm to (57.8, 34.9), turned to 270 degrees
- moved C4 5.12 mm to (62.2, 34.9), turned to 270 degrees
- moved D2 5.08 mm to (113.1, 60.7)
- moved R1 2.29 mm to (112.9, 20.4)
- moved C1 2.29 mm to (70.6, 37.1)
- moved C6 2.04 mm to (66.0, 45.1), turned to 90 degrees
- moved J5 1.80 mm to (103.6, 80.4)
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Connections:
- removed net N$69: J4.23, U3.99
- removed net N$70: J4.21, U3.97
- removed net N$71: J4.19, U3.95
- removed net N$72: J4.17, U3.93
- removed net N$73: J4.15, U3.91
- removed net N$74: J4.13, U3.89
- removed net N$75: J4.11, U3.87
- new net RA6: J16.9, J4.15, U3.91
- new net RE0: J16.7, J4.17, U3.93
- new net RE3: J16.1, J4.23, U3.99
- new net RF0: J16.13, J4.11, U3.87
- new net RG1: J16.11, J4.13, U3.89
- new net RG13: J16.3, J4.21, U3.97
- new net RG14: J16.5, J4.19, U3.95
- net +3V3: now also J14.3, J15.1, J16.10, J16.12, J16.14, R4.2, R5.2
- net GND: now also J14.1, J15.4, J16.2, J16.4, J16.6, J16.8
- net N$26: now also R6.2
- net N$28: now also R6.1
- net N$8: now also J14.2
- net SCL1: now also J15.2
- net SDA1: now also J15.3
- net SD_CS: now also CS.P$1
- net SD_MISO: now also MISO.P$1
- net SD_MOSI: now also MOSI.P$1
- net SD_SCK: now also SCK.P$1
- net U1RX: now also R5.1
- net U1TX: now also R4.1
Routing:
- net +3V3: track 511.9 -> 581.4 mm
- net RE3: track 0.00 -> 56.8 mm
- net RG13: track 0.00 -> 55.8 mm
- net RG14: track 0.00 -> 54.4 mm
- net RE0: track 0.00 -> 52.5 mm
- net RA6: track 0.00 -> 50.8 mm
- net RG1: track 0.00 -> 50.0 mm
- net RF0: track 0.00 -> 48.5 mm
- net N$69: track 43.1 -> 0.00 mm
- net N$8: track 20.5 -> 63.4 mm
- net N$70: track 41.5 -> 0.00 mm
- net N$71: track 40.8 -> 0.00 mm
- net N$72: track 39.7 -> 0.00 mm
- net N$73: track 38.7 -> 0.00 mm
- net N$74: track 37.4 -> 0.00 mm
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Other:
- board text added: "A"
- board text added: "B"
- board text added: "G"
- board text added: "OC3"
- board text added: "OC5"
- board text added: "PORT B"
- board text added: "SCL1"
- board text added: "SCL3"
- board text added: "SDA1"
- board text added: "SDA3"
- board text added: "T1CK"
- board text added: "U4TX"
- board text removed: "ANALOG IN"
- board text removed: "OC1/RD0/SDO1"
- board text removed: "OC3/RD2"
- board text removed: "OC5/RD4"
- board text removed: "RB12"
- board text removed: "RB14"
- board text removed: "RD15/U4TX"
- board text removed: "RD8"
- board text removed: "RF13"
- board text removed: "RS485"
- board text removed: "SCK1/RD10"
- board text removed: "SCL1/RA14"
- board text removed: "T1CK/RC14"
- board text removed: "UART 1"
