File: PIC795 Brain Board.sch (EAGLE design)
At the start: 56 parts, among them J10 MOLEX_4PMOLEX_4P, J11 MOLEX_6P, J12 MOLEX_3P, J13 MOLEX-2P-156, J5 MOLEX_4PMOLEX_4P, J6 MOLEX_4PMOLEX_4P, J7 USB+SHIELD, J8 POWER_JACK, J9 RJ11-2L-B, SW1 E_SWITCH-320, U1 REGULATOR_LD1086_LDO, U2 SD_CARD, U3 PIC32MX795F512L, U4 MAX4830, U5 24LC256, X1 8 Mhz

Commit message: Add files via upload
Minor changes for Rev 2
Parts:
- D1, D2: value 1N5817-B -> 40V
- LED1: value (none) -> RED
- LED2: value (none) -> YELLOW
- R1, R3: value 120 ohm -> 220 ohm
Connections:
- net !SD_CS renamed T5CK
- net GND: no longer J1.25, J1.26
Other:
- note added: "2"
- note removed: "2.0"
Changed lines of the file:
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@@
 <part name="GND10" library="supply1" deviceset="GND" device=""/>
 <part name="GND11" library="supply1" deviceset="GND" device=""/>
-<part name="R1" library="JimLib" deviceset="RESISTOR" device="0207/12" value="120 ohm"/>
-<part name="LED1" library="JimLib" deviceset="LED" device="5MM"/>
+<part name="R1" library="JimLib" deviceset="RESISTOR" device="0207/12" value="220 ohm"/>
+<part name="LED1" library="JimLib" deviceset="LED" device="5MM" value="RED"/>
 <part name="GND22" library="supply1" deviceset="GND" device=""/>
 <part name="+3V9" library="supply1" deviceset="+3V3" device=""/>
@@
 <part name="C14" library="JimLib" deviceset="POLCAP" device="E2.5-5" value="10 uF"/>
 <part name="U1" library="JimLib" deviceset="REGULATOR_LD1086_LDO" device=""/>
-<part name="D1" library="JimLib" deviceset="1N581*" device="" technology="7-B"/>
+<part name="D1" library="JimLib" deviceset="1N581*" device="" technology="7-B" value="40V"/>
 <part name="U2" library="JimLib" deviceset="SD_CARD" device=""/>
 <part name="J8" library="JimLib" deviceset="POWER_JACK" device=""/>
@@
 <part name="+3V18" library="supply1" deviceset="+3V3" device=""/>
 <part name="GND3" library="supply1" deviceset="GND" device=""/>
-<part name="GND30" library="supply1" deviceset="GND" device=""/>
 <part name="+3V19" library="supply1" deviceset="+3V3" device=""/>
 <part name="+3V20" library="supply1" deviceset="+3V3" device=""/>
@@
 <part name="GND32" library="supply1" deviceset="GND" device=""/>
 <part name="GND33" library="supply1" deviceset="GND" device=""/>
-<part name="D2" library="JimLib" deviceset="1N581*" device="" technology="7-B"/>
+<part name="D2" library="JimLib" deviceset="1N581*" device="" technology="7-B" value="40V"/>
 <part name="U5" library="JimLib" deviceset="EEPROM_24LC256" device="" value="24LC256"/>
 <part name="+3V21" library="supply1" deviceset="+3V3" device=""/>
@@
 <part name="J13" library="JimLib" deviceset="MOLEX-2P-156" device=""/>
 <part name="GND35" library="supply1" deviceset="GND" device=""/>
-<part name="LED2" library="JimLib" deviceset="LED" device="5MM"/>
-<part name="R3" library="JimLib" deviceset="RESISTOR" device="0207/12" value="120 ohm"/>
+<part name="LED2" library="JimLib" deviceset="LED" device="5MM" value="YELLOW"/>
+<part name="R3" library="JimLib" deviceset="RESISTOR" device="0207/12" value="220 ohm"/>
 <part name="GND36" library="supply1" deviceset="GND" device=""/>
 <part name="TEST_OUT" library="JimLib" deviceset="TP" device=""/>
@@
 <sheet>
 <plain>
-<text x="165.1" y="-45.72" size="1.778" layer="94">2.0</text>
+<text x="166.37" y="-46.99" size="3.81" layer="94">2</text>
 </plain>
 <instances>
@@
 <instance part="+3V18" gate="G$1" x="-104.14" y="77.47"/>
 <instance part="GND3" gate="1" x="-229.87" y="171.45"/>
-<instance part="GND30" gate="1" x="-224.79" y="129.54"/>
 <instance part="+3V19" gate="G$1" x="13.97" y="177.8"/>
 <instance part="+3V20" gate="G$1" x="-24.13" y="168.91" rot="R90"/>
@@
 </segment>
 </net>
-<net name="!SD_CS" class="0">
+<net name="T5CK" class="0">
 <segment>
 <wire x1="-154.94" y1="175.26" x2="-189.23" y2="175.26" width="0.1524" layer="91"/>
@@
 <wire x1="-285.75" y1="290.83" x2="-275.59" y2="290.83" width="0.1524" layer="91"/>
 <wire x1="-275.59" y1="290.83" x2="-275.59" y2="300.99" width="0.1524" layer="91"/>
+<junction x="-275.59" y="300.99"/>
 </segment>
 </net>
@@
 </segment>
 <segment>
-<pinref part="J1" gate="G$1" pin="25"/>
-<wire x1="-209.55" y1="146.05" x2="-224.79" y2="146.05" width="0.1524" layer="91"/>
-<wire x1="-224.79" y1="146.05" x2="-224.79" y2="139.7" width="0.1524" layer="91"/>
-<pinref part="GND30" gate="1" pin="GND"/>
-<pinref part="J1" gate="G$1" pin="26"/>
-<wire x1="-194.31" y1="146.05" x2="-194.31" y2="139.7" width="0.1524" layer="91"/>
-<wire x1="-194.31" y1="139.7" x2="-224.79" y2="139.7" width="0.1524" layer="91"/>
-<wire x1="-224.79" y1="139.7" x2="-224.79" y2="132.08" width="0.1524" layer="91"/>
-<junction x="-224.79" y="139.7"/>
-</segment>
-<segment>

Commit message: Add files via upload
Includes latest changes for Rev 2. Shipped to PCB fab 8-12-19
Parts:
- added CS, MISO, MOSI, SCK: TP, JimLib:TP
- added J14: MOLEX_MINI_RA_3P, JimLib:MOLEX_MINI_RA_3P
- added J15: MOLEX_4PMOLEX_4P, JimLib:MOLEX_4PMOLEX_4P
- added J16: (no value), JimLib:CONNECTOR_DUAL_ROW_14
- added R4, R5: 10K, JimLib:RESISTOR0207/12
- added R6: 180 ohms, JimLib:RESISTOR0204/7
Connections:
- removed net N$69: J4.23, U3.RE3
- removed net N$70: J4.21, U3.RG13
- removed net N$71: J4.19, U3.RG14
- removed net N$72: J4.17, U3.RE0
- removed net N$73: J4.15, U3.RA6
- removed net N$74: J4.13, U3.RG1
- removed net N$75: J4.11, U3.RF0
- new net RA6: J16.9, J4.15, U3.RA6
- new net RE0: J16.7, J4.17, U3.RE0
- new net RE3: J16.1, J4.23, U3.RE3
- new net RF0: J16.13, J4.11, U3.RF0
- new net RG1: J16.11, J4.13, U3.RG1
- new net RG13: J16.3, J4.21, U3.RG13
- new net RG14: J16.5, J4.19, U3.RG14
- net +3V3: now also J14.3, J15.1, J16.10, J16.12, J16.14, R4.2, R5.2
- net GND: now also J14.1, J15.4, J16.2, J16.4, J16.6, J16.8
- net N$26: now also R6.2
- net N$28: now also R6.1
- net N$8: now also J14.2
- net SCL1: now also J15.2
- net SDA1: now also J15.3
- net SD_CS: now also CS.TP
- net SD_MISO: now also MISO.TP
- net SD_MOSI: now also MOSI.TP
- net SD_SCK: now also SCK.TP
- net U1RX: now also R5.1
- net U1TX: now also R4.1
Other:
- note added: "+3.3V"
- note added: "GND"
- note added: "SCL1"
- note added: "SCL3"
- note added: "SDA1"
- note added: "SDA3"
- moved on the sheet: J12, J5
